Commit message: Added example robots

File: inovo_description/urdf/examples/prd_long.urdf (robot description, URDF)
Before this commit: robot autogen-robot, 12 links, 6 joints
Links:
- removed link joint_prdlink1
- added link joint_prdlink2, mass 1.084; collision cylinder length=0.33 radius=0.05; visual mesh filename=package://inovo_description/meshes/prd/TUBE_300.dae
- added link joint_prdlink3, mass 1.321; collision cylinder length=0.473 radius=0.05; visual mesh filename=package://inovo_description/meshes/prd/TUBE_470.dae
Joints:
- removed joint joint_prdlink1_coupling
- added joint joint_prdlink2_coupling: type fixed, parent joint_prdlink2, child joint_elbow_output, origin xyz=0 0 0.3004 rpy=0 0 0
- added joint joint_prdlink3_coupling: type fixed, parent joint_prdlink3, child joint_shoulder, origin xyz=0 0 0.4704 rpy=0 0 0

File: inovo_description/urdf/examples/prd_medium.urdf (robot description, URDF)
Before this commit: robot autogen-robot, 12 links, 6 joints
Links:
- added link joint_prdlink2, mass 1.084; collision cylinder length=0.33 radius=0.05; visual mesh filename=package://inovo_description/meshes/prd/TUBE_300.dae
Joints:
- added joint joint_prdlink2_coupling: type fixed, parent joint_prdlink2, child joint_shoulder, origin xyz=0 0 0.3004 rpy=0 0 0
- joint joint_prdlink1_coupling: child joint_shoulder -> joint_elbow_output

Commit message: Updated example urdfs and added inovo_viz package

File: inovo_description/urdf/examples/prd_long.urdf (robot description, URDF)
Before this commit: robot autogen-robot, 13 links, 7 joints
Links:
- removed link joint_base
- removed link joint_elbow
- removed link joint_elbow_output
- removed link joint_forearm
- removed link joint_jlink
- removed link joint_prd1192
- removed link joint_prdlink2
- removed link joint_prdlink3
- removed link joint_shoulder
- removed link joint_shoulder_output
- removed link joint_wrist_b
- added link j1_base, mass 4.696; collision cylinder length=0.18 radius=0.08; visual mesh filename=package://inovo_description/meshes/prd/J1.dae
- added link j2_shoulder, mass 5.24; collision cylinder length=0.17 radius=0.08; visual mesh filename=package://inovo_description/meshes/prd/J2.dae
- added link j2_shoulder_output, mass 2.243; collision cylinder length=0.11 radius=0.08; visual mesh filename=package://inovo_description/meshes/prd/J2_1.dae
- added link j3_prdlink3, mass 1.321; collision cylinder length=0.473 radius=0.05; visual mesh filename=package://inovo_description/meshes/prd/TUBE_470.dae
- added link j4_elbow, mass 2.58; collision cylinder length=0.14 radius=0.06; visual mesh filename=package://inovo_description/meshes/prd/J3.dae
- added link j5_elbow_output, mass 2.582; collision cylinder length=0.15 radius=0.06; visual mesh filename=package://inovo_description/meshes/prd/J4.dae
- added link j5_forearm, mass 0.686; collision cylinder length=0.025 radius=0.06; visual mesh filename=package://inovo_description/meshes/prd/J4_1.dae
- added link j6_prdlink2, mass 1.084; collision cylinder length=0.33 radius=0.05; visual mesh filename=package://inovo_description/meshes/prd/TUBE_300.dae
- added link j7_jlink, mass 2.187; collision mesh filename=package://inovo_description/meshes/prd/J5_collision.stl; visual mesh filename=package://inovo_description/meshes/prd/J5.dae
- added link j8_prd1192, mass 0.38; collision cylinder length=0.035 radius=0.045; visual mesh filename=package://inovo_description/meshes/prd/J6_1.dae
- added link j8_wrist_b, mass 1.933; collision cylinder length=0.14 radius=0.045; visual mesh filename=package://inovo_description/meshes/prd/J6.dae
Joints:
- removed joint joint
- removed joint joint_forearm_coupling
- removed joint joint_prd1190_fixed
- removed joint joint_prdlink2_coupling
- removed joint joint_prdlink3_coupling
- removed joint joint_shoulder_output_joint
- added joint j1: type continuous, parent j1_base, child j2_shoulder, origin xyz=0 0 0.26022 rpy=0 0 0, axis 0 0 1, limit effort=3.0 velocity=1.8
- added joint j2: type continuous, parent j2_shoulder, child j2_shoulder_output, origin xyz=0.1335 0 0 rpy=0 4.7123889804 3.14159265359, axis 0 0 1, limit effort=4.0 velocity=1.8
- added joint j2_shoulder_output_joint: type fixed, parent j2_shoulder_output, child j3_prdlink3, origin xyz=0.07975 0.0 0.0 rpy=3.14159265359 -1.57079632679 0
- added joint j3_prdlink3_coupling: type fixed, parent j3_prdlink3, child j4_elbow, origin xyz=0 0 0.4704 rpy=0 0 0
- added joint j4: type continuous, parent j4_elbow, child j5_elbow_output, origin xyz=0 0 0.09025 rpy=0 -1.57079632679 0, axis 0 0 1, limit effort=10.0 velocity=2.5
- added joint j5: type continuous, parent j5_elbow_output, child j5_forearm, origin xyz=0 0 0.1335 rpy=0 -1.57079632679 3.141592653590, axis 0 0 1, limit effort=10.0 velocity=2.6
- added joint j5_forearm_coupling: type fixed, parent j5_forearm, child j6_prdlink2, origin xyz=0 0 0.09477 rpy=0 0 3.141592653590
- added joint j6_prdlink2_coupling: type fixed, parent j6_prdlink2, child j7_jlink, origin xyz=0 0 0.3004 rpy=0 0 0
- added joint j7: type continuous, parent j7_jlink, child j8_wrist_b, origin xyz=0 0 0.30523 rpy=0 -1.5707963267908 0, axis 0 0 1, limit effort=20.0 velocity=3.3
- added joint j8: type continuous, parent j8_wrist_b, child j8_prd1192, origin xyz=0 0 0.0 rpy=0 -1.5707963267908 3.141592653590, axis 0 0 1, limit effort=25.0 velocity=3.3
- added joint j8_prd1190_fixed: type fixed, parent j8_prd1192, child flange, origin xyz=0 0 0.0926 rpy=0 0 0
- joint world: child joint_wrist_b -> j1_base

File: inovo_description/urdf/examples/prd_medium.urdf (robot description, URDF)
Before this commit: robot autogen-robot, 13 links, 7 joints
Links:
- removed link joint_base
- removed link joint_elbow
- removed link joint_elbow_output
- removed link joint_forearm
- removed link joint_jlink
- removed link joint_prd1192
- removed link joint_prdlink1
- removed link joint_prdlink2
- removed link joint_shoulder
- removed link joint_shoulder_output
- removed link joint_wrist_b
- added link j1_base, mass 4.696; collision cylinder length=0.18 radius=0.08; visual mesh filename=package://inovo_description/meshes/prd/J1.dae
- added link j2_shoulder, mass 5.24; collision cylinder length=0.17 radius=0.08; visual mesh filename=package://inovo_description/meshes/prd/J2.dae
- added link j2_shoulder_output, mass 2.243; collision cylinder length=0.11 radius=0.08; visual mesh filename=package://inovo_description/meshes/prd/J2_1.dae
- added link j3_prdlink2, mass 1.084; collision cylinder length=0.33 radius=0.05; visual mesh filename=package://inovo_description/meshes/prd/TUBE_300.dae
- added link j4_elbow, mass 2.58; collision cylinder length=0.14 radius=0.06; visual mesh filename=package://inovo_description/meshes/prd/J3.dae
- added link j5_elbow_output, mass 2.582; collision cylinder length=0.15 radius=0.06; visual mesh filename=package://inovo_description/meshes/prd/J4.dae
- added link j5_forearm, mass 0.686; collision cylinder length=0.025 radius=0.06; visual mesh filename=package://inovo_description/meshes/prd/J4_1.dae
- added link j6_prdlink1, mass 0.834; collision cylinder length=0.14 radius=0.06; visual mesh filename=package://inovo_description/meshes/prd/TUBE_120.dae
- added link j7_jlink, mass 2.187; collision mesh filename=package://inovo_description/meshes/prd/J5_collision.stl; visual mesh filename=package://inovo_description/meshes/prd/J5.dae
- added link j8_prd1192, mass 0.38; collision cylinder length=0.035 radius=0.045; visual mesh filename=package://inovo_description/meshes/prd/J6_1.dae
- added link j8_wrist_b, mass 1.933; collision cylinder length=0.14 radius=0.045; visual mesh filename=package://inovo_description/meshes/prd/J6.dae
Joints:
- removed joint joint
- removed joint joint_forearm_coupling
- removed joint joint_prd1190_fixed
- removed joint joint_prdlink1_coupling
- removed joint joint_prdlink2_coupling
- removed joint joint_shoulder_output_joint
- added joint j1: type continuous, parent j1_base, child j2_shoulder, origin xyz=0 0 0.26022 rpy=0 0 0, axis 0 0 1, limit effort=3.0 velocity=1.8
- added joint j2: type continuous, parent j2_shoulder, child j2_shoulder_output, origin xyz=0.1335 0 0 rpy=0 4.7123889804 3.14159265359, axis 0 0 1, limit effort=4.0 velocity=1.8
- added joint j2_shoulder_output_joint: type fixed, parent j2_shoulder_output, child j3_prdlink2, origin xyz=0.07975 0.0 0.0 rpy=3.14159265359 -1.57079632679 0
- added joint j3_prdlink2_coupling: type fixed, parent j3_prdlink2, child j4_elbow, origin xyz=0 0 0.3004 rpy=0 0 0
- added joint j4: type continuous, parent j4_elbow, child j5_elbow_output, origin xyz=0 0 0.09025 rpy=0 -1.57079632679 0, axis 0 0 1, limit effort=10.0 velocity=2.5
- added joint j5: type continuous, parent j5_elbow_output, child j5_forearm, origin xyz=0 0 0.1335 rpy=0 -1.57079632679 3.141592653590, axis 0 0 1, limit effort=10.0 velocity=2.6
- added joint j5_forearm_coupling: type fixed, parent j5_forearm, child j6_prdlink1, origin xyz=0 0 0.09477 rpy=0 0 3.141592653590
- added joint j6_prdlink1_coupling: type fixed, parent j6_prdlink1, child j7_jlink, origin xyz=0 0 0.1196 rpy=0 0 0
- added joint j7: type continuous, parent j7_jlink, child j8_wrist_b, origin xyz=0 0 0.30523 rpy=0 -1.5707963267908 0, axis 0 0 1, limit effort=20.0 velocity=3.3
- added joint j8: type continuous, parent j8_wrist_b, child j8_prd1192, origin xyz=0 0 0.0 rpy=0 -1.5707963267908 3.141592653590, axis 0 0 1, limit effort=25.0 velocity=3.3
- added joint j8_prd1190_fixed: type fixed, parent j8_prd1192, child flange, origin xyz=0 0 0.0926 rpy=0 0 0
- joint world: child joint_wrist_b -> j1_base

File: inovo_description/urdf/examples/prd_short.urdf (robot description, URDF)
Before this commit: robot autogen-robot, 12 links, 6 joints
Links:
- removed link joint_base
- removed link joint_elbow
- removed link joint_elbow_output
- removed link joint_forearm
- removed link joint_jlink
- removed link joint_prd1192
- removed link joint_prdlink1
- removed link joint_shoulder
- removed link joint_shoulder_output
- removed link joint_wrist_b
- added link j1_base, mass 4.696; collision cylinder length=0.18 radius=0.08; visual mesh filename=package://inovo_description/meshes/prd/J1.dae
- added link j2_shoulder, mass 5.24; collision cylinder length=0.17 radius=0.08; visual mesh filename=package://inovo_description/meshes/prd/J2.dae
- added link j2_shoulder_output, mass 2.243; collision cylinder length=0.11 radius=0.08; visual mesh filename=package://inovo_description/meshes/prd/J2_1.dae
- added link j3_prdlink1, mass 0.834; collision cylinder length=0.14 radius=0.06; visual mesh filename=package://inovo_description/meshes/prd/TUBE_120.dae
- added link j4_elbow, mass 2.58; collision cylinder length=0.14 radius=0.06; visual mesh filename=package://inovo_description/meshes/prd/J3.dae
- added link j5_elbow_output, mass 2.582; collision cylinder length=0.15 radius=0.06; visual mesh filename=package://inovo_description/meshes/prd/J4.dae
- added link j5_forearm, mass 0.686; collision cylinder length=0.025 radius=0.06; visual mesh filename=package://inovo_description/meshes/prd/J4_1.dae
- added link j6_jlink, mass 2.187; collision mesh filename=package://inovo_description/meshes/prd/J5_collision.stl; visual mesh filename=package://inovo_description/meshes/prd/J5.dae
- added link j7_prd1192, mass 0.38; collision cylinder length=0.035 radius=0.045; visual mesh filename=package://inovo_description/meshes/prd/J6_1.dae
- added link j7_wrist_b, mass 1.933; collision cylinder length=0.14 radius=0.045; visual mesh filename=package://inovo_description/meshes/prd/J6.dae
Joints:
- removed joint joint
- removed joint joint_forearm_coupling
- removed joint joint_prd1190_fixed
- removed joint joint_prdlink1_coupling
- removed joint joint_shoulder_output_joint
- added joint j1: type continuous, parent j1_base, child j2_shoulder, origin xyz=0 0 0.26022 rpy=0 0 0, axis 0 0 1, limit effort=3.0 velocity=1.8
- added joint j2: type continuous, parent j2_shoulder, child j2_shoulder_output, origin xyz=0.1335 0 0 rpy=0 4.7123889804 3.14159265359, axis 0 0 1, limit effort=4.0 velocity=1.8
- added joint j2_shoulder_output_joint: type fixed, parent j2_shoulder_output, child j3_prdlink1, origin xyz=0.07975 0.0 0.0 rpy=3.14159265359 -1.57079632679 0
- added joint j3_prdlink1_coupling: type fixed, parent j3_prdlink1, child j4_elbow, origin xyz=0 0 0.1196 rpy=0 0 0
- added joint j4: type continuous, parent j4_elbow, child j5_elbow_output, origin xyz=0 0 0.09025 rpy=0 -1.57079632679 0, axis 0 0 1, limit effort=10.0 velocity=2.5
- added joint j5: type continuous, parent j5_elbow_output, child j5_forearm, origin xyz=0 0 0.1335 rpy=0 -1.57079632679 3.141592653590, axis 0 0 1, limit effort=10.0 velocity=2.6
- added joint j5_forearm_coupling: type fixed, parent j5_forearm, child j6_jlink, origin xyz=0 0 0.09477 rpy=0 0 3.141592653590
- added joint j6: type continuous, parent j6_jlink, child j7_wrist_b, origin xyz=0 0 0.30523 rpy=0 -1.5707963267908 0, axis 0 0 1, limit effort=20.0 velocity=3.3
- added joint j7: type continuous, parent j7_wrist_b, child j7_prd1192, origin xyz=0 0 0.0 rpy=0 -1.5707963267908 3.141592653590, axis 0 0 1, limit effort=25.0 velocity=3.3
- added joint j7_prd1190_fixed: type fixed, parent j7_prd1192, child flange, origin xyz=0 0 0.0926 rpy=0 0 0
- joint world: child joint_wrist_b -> j1_base
