Commit message: Updated medium prd urdf example to be much more readable and added the correct effort limits

File: inovo_description/urdf/examples/prd_medium.urdf (robot description, URDF)
Before this commit: robot inovo_robot, 13 links, 12 joints
Links:
- removed link j1_base
- removed link j2_shoulder
- removed link j2_shoulder_output
- removed link j3_prdlink2
- removed link j4_elbow
- removed link j5_elbow_output
- removed link j5_forearm
- removed link j6_prdlink1
- removed link j7_jlink
- removed link j8_prd1192
- removed link j8_wrist_b
- removed link world
- added link base, mass 4.696; collision cylinder length=0.18 radius=0.08; visual mesh filename=package://inovo_description/meshes/prd/J1.dae
- added link elbow, mass 2.58; collision cylinder length=0.14 radius=0.06; visual mesh filename=package://inovo_description/meshes/prd/J3.dae
- added link forearm, mass 0.834; collision cylinder length=0.14 radius=0.06; visual mesh filename=package://inovo_description/meshes/prd/TUBE_120.dae
- added link shoulder, mass 5.24; collision cylinder length=0.17 radius=0.08; visual mesh filename=package://inovo_description/meshes/prd/J2.dae
- added link shoulder_output, mass 2.243; collision cylinder length=0.11 radius=0.08; visual mesh filename=package://inovo_description/meshes/prd/J2_1.dae
- added link upper_arm_link, mass 1.084; collision cylinder length=0.33 radius=0.05; visual mesh filename=package://inovo_description/meshes/prd/TUBE_300.dae
- added link wrist_a, mass 2.582; collision cylinder length=0.15 radius=0.06; visual mesh filename=package://inovo_description/meshes/prd/J4.dae
- added link wrist_a_output, mass 0.686; collision cylinder length=0.025 radius=0.06; visual mesh filename=package://inovo_description/meshes/prd/J4_1.dae
- added link wrist_b, mass 2.187; collision mesh filename=package://inovo_description/meshes/prd/J5_collision.stl; visual mesh filename=package://inovo_description/meshes/prd/J5.dae
- added link wrist_c, mass 1.933; collision cylinder length=0.14 radius=0.045; visual mesh filename=package://inovo_description/meshes/prd/J6.dae
- added link wrist_c_output, mass 0.38; collision cylinder length=0.035 radius=0.045; visual mesh filename=package://inovo_description/meshes/prd/J6_1.dae
Joints:
- removed joint j2_shoulder_output_joint
- removed joint j3_prdlink2_coupling
- removed joint j5_forearm_coupling
- removed joint j6_prdlink1_coupling
- removed joint j7
- removed joint j8
- removed joint j8_prd1190_fixed
- removed joint world
- added joint flange_coupling: type fixed, parent wrist_c_output, child flange, origin xyz=0 0 0.0926 rpy=0 0 0
- added joint forearm_coupling: type fixed, parent forearm, child wrist_b, origin xyz=0 0 0.1196 rpy=0 0 0
- added joint j3: type continuous, parent elbow, child wrist_a, origin xyz=0 0 0.09025 rpy=0 -1.57079632679 0, axis 0 0 1, limit effort=10.0 velocity=2.5
- added joint j6: type continuous, parent wrist_c, child wrist_c_output, origin xyz=0 0 0.0 rpy=0 -1.5707963267908 3.141592653590, axis 0 0 1, limit effort=25.0 velocity=3.3
- added joint shoulder_output_coupling: type fixed, parent shoulder_output, child upper_arm_link, origin xyz=0.07975 0.0 0.0 rpy=3.14159265359 -1.57079632679 0
- added joint upper_arm_coupling: type fixed, parent upper_arm_link, child elbow, origin xyz=0 0 0.3004 rpy=0 0 0
- added joint wrist_a_output_coupling: type fixed, parent wrist_a_output, child forearm, origin xyz=0 0 0.09477 rpy=0 0 3.141592653590
- joint j1: child j2_shoulder -> shoulder; parent j1_base -> base
- joint j2: child j2_shoulder_output -> shoulder_output; parent j2_shoulder -> shoulder
- joint j4: child j5_elbow_output -> wrist_a_output; limit effort=10.0 velocity=2.5 -> effort=10.0 velocity=2.6; origin xyz=0 0 0.09025 rpy=0 -1.57079632679 0 -> xyz=0 0 0.1335 rpy=0 -1.57079632679 3.141592653590; parent j4_elbow -> wrist_a
- joint j5: child j5_forearm -> wrist_c; limit effort=10.0 velocity=2.6 -> effort=20.0 velocity=3.3; origin xyz=0 0 0.1335 rpy=0 -1.57079632679 3.141592653590 -> xyz=0 0 0.30523 rpy=0 -1.5707963267908 0; parent j5_elbow_output -> wrist_b
